File: _autosave-tracker.sch (KiCad schematic (older format))
At the start: 46 parts, among them J1 USB_C_Receptacle_USB2.0, J2 BAT, Q1 UMH3N, SW1 SW_Push, SW2 PWR_SW, U1 TP4056, U2 BNO055, U3 CH340C, U4 DW01, U5 FS8205A, U6 ESP-12F, U7 TPS63001, Y1 32.768 Khz

Commit message: REV1.1
Parts:
- L1: footprint Inductor_SMD:L_2816_7142Metric_Pad3.20x4.45mm_HandSolder -> Inductor_SMD:L_1210_3225Metric_Pad1.42x2.65mm_HandSolder
Changed lines of the file:
@@
 F 0 "L1" H 9250 4965 50  0000 C CNN
 F 1 "2.2uH" H 9250 4874 50  0000 C CNN
-F 2 "Inductor_SMD:L_2816_7142Metric_Pad3.20x4.45mm_HandSolder" H 9250 4750 50  0001 C CNN
+F 2 "Inductor_SMD:L_1210_3225Metric_Pad1.42x2.65mm_HandSolder" H 9250 4750 50  0001 C CNN
 F 3 "~" H 9250 4750 50  0001 C CNN
 	1    9250 4750

Commit message: metric/imperial fix
Parts:
- C1, C10, C2, C3, C4, C5, C6, C7, C8, C9: footprint Capacitor_SMD:C_0201_0603Metric_Pad0.64x0.40mm_HandSolder -> Resistor_SMD:R_0402_1005Metric_Pad0.72x0.64mm_HandSolder
- R1, R10, R11, R12, R13, R14, R15, R16, R17, R18, R19, R2, R20, R3, R4, R5, R6, R7, R8, R9: footprint Resistor_SMD:R_0201_0603Metric_Pad0.64x0.40mm_HandSolder -> Resistor_SMD:R_0402_1005Metric_Pad0.72x0.64mm_HandSolder
Changed lines of the file:
@@
 F 0 "C2" V 4500 2450 50  0000 C CNN
 F 1 "0.1 uF" V 4400 2450 50  0000 C CNN
-F 2 "Capacitor_SMD:C_0201_0603Metric_Pad0.64x0.40mm_HandSolder" H 4200 2450 50  0001 C CNN
+F 2 "Resistor_SMD:R_0402_1005Metric_Pad0.72x0.64mm_HandSolder" H 4200 2450 50  0001 C CNN
 F 3 "~" H 4200 2450 50  0001 C CNN
 	1    4200 2450
@@
 F 0 "R2" H 2220 1846 50  0000 L CNN
 F 1 "10K" H 2220 1755 50  0000 L CNN
-F 2 "Resistor_SMD:R_0201_0603Metric_Pad0.64x0.40mm_HandSolder" V 2080 1800 50  0001 C CNN
+F 2 "Resistor_SMD:R_0402_1005Metric_Pad0.72x0.64mm_HandSolder" V 2080 1800 50  0001 C CNN
 F 3 "~" H 2150 1800 50  0001 C CNN
 	1    2150 1800
@@
 F 0 "R1" H 1920 1846 50  0000 L CNN
 F 1 "10K" H 1920 1755 50  0000 L CNN
-F 2 "Resistor_SMD:R_0201_0603Metric_Pad0.64x0.40mm_HandSolder" V 1780 1800 50  0001 C CNN
+F 2 "Resistor_SMD:R_0402_1005Metric_Pad0.72x0.64mm_HandSolder" V 1780 1800 50  0001 C CNN
 F 3 "~" H 1850 1800 50  0001 C CNN
 	1    1850 1800
@@
 F 0 "R6" V 2550 2300 50  0000 C CNN
 F 1 "10K" V 2450 2300 50  0000 C CNN
-F 2 "Resistor_SMD:R_0201_0603Metric_Pad0.64x0.40mm_HandSolder" V 2280 2300 50  0001 C CNN
+F 2 "Resistor_SMD:R_0402_1005Metric_Pad0.72x0.64mm_HandSolder" V 2280 2300 50  0001 C CNN
 F 3 "~" H 2350 2300 50  0001 C CNN
 	1    2350 2300
@@
 F 0 "R5" V 2100 1300 50  0000 C CNN
 F 1 "10K" V 2200 1300 50  0000 C CNN
-F 2 "Resistor_SMD:R_0201_0603Metric_Pad0.64x0.40mm_HandSolder" V 2230 1300 50  0001 C CNN
+F 2 "Resistor_SMD:R_0402_1005Metric_Pad0.72x0.64mm_HandSolder" V 2230 1300 50  0001 C CNN
 F 3 "~" H 2300 1300 50  0001 C CNN
 	1    2300 1300
@@
 F 0 "R11" V 4050 2400 50  0000 C CNN
 F 1 "10K" V 4050 2000 50  0000 C CNN
-F 2 "Resistor_SMD:R_0201_0603Metric_Pad0.64x0.40mm_HandSolder" V 4030 2200 50  0001 C CNN
+F 2 "Resistor_SMD:R_0402_1005Metric_Pad0.72x0.64mm_HandSolder" V 4030 2200 50  0001 C CNN
 F 3 "~" H 4100 2200 50  0001 C CNN
 	1    4100 2200
@@
 F 0 "R10" V 4050 2300 50  0000 C CNN
 F 1 "10K" V 4050 1900 50  0000 C CNN
-F 2 "Resistor_SMD:R_0201_0603Metric_Pad0.64x0.40mm_HandSolder" V 4030 2100 50  0001 C CNN
+F 2 "Resistor_SMD:R_0402_1005Metric_Pad0.72x0.64mm_HandSolder" V 4030 2100 50  0001 C CNN
 F 3 "~" H 4100 2100 50  0001 C CNN
 	1    4100 2100
@@
 F 0 "C4" V 4350 1450 50  0000 C CNN
 F 1 "22 pF" V 4350 1100 50  0000 C CNN
-F 2 "Capacitor_SMD:C_0201_0603Metric_Pad0.64x0.40mm_HandSolder" H 4450 1300 50  0001 C CNN
+F 2 "Resistor_SMD:R_0402_1005Metric_Pad0.72x0.64mm_HandSolder" H 4450 1300 50  0001 C CNN
 F 3 "~" H 4450 1300 50  0001 C CNN
 	1    4450 1300
@@
 F 0 "C5" V 4350 1950 50  0000 C CNN
 F 1 "22 pF" V 4350 1600 50  0000 C CNN
-F 2 "Capacitor_SMD:C_0201_0603Metric_Pad0.64x0.40mm_HandSolder" H 4450 1800 50  0001 C CNN
+F 2 "Resistor_SMD:R_0402_1005Metric_Pad0.72x0.64mm_HandSolder" H 4450 1800 50  0001 C CNN
 F 3 "~" H 4450 1800 50  0001 C CNN
 	1    4450 1800
@@
 F 0 "R7" V 2900 3900 50  0000 C CNN
 F 1 "5.1K" V 2900 3500 50  0000 C CNN
-F 2 "Resistor_SMD:R_0201_0603Metric_Pad0.64x0.40mm_HandSolder" V 2880 3700 50  0001 C CNN
+F 2 "Resistor_SMD:R_0402_1005Metric_Pad0.72x0.64mm_HandSolder" V 2880 3700 50  0001 C CNN
 F 3 "~" H 2950 3700 50  0001 C CNN
 	1    2950 3700
@@
 F 0 "R8" V 2900 4000 50  0000 C CNN
 F 1 "5.1K" V 2900 3600 50  0000 C CNN
-F 2 "Resistor_SMD:R_0201_0603Metric_Pad0.64x0.40mm_HandSolder" V 2880 3800 50  0001 C CNN
+F 2 "Resistor_SMD:R_0402_1005Metric_Pad0.72x0.64mm_HandSolder" V 2880 3800 50  0001 C CNN
 F 3 "~" H 2950 3800 50  0001 C CNN
 	1    2950 3800
@@
 F 0 "R3" V 2300 6750 50  0000 L CNN
 F 1 "1K" V 2300 6350 50  0000 L CNN
-F 2 "Resistor_SMD:R_0201_0603Metric_Pad0.64x0.40mm_HandSolder" V 2180 6600 50  0001 C CNN
+F 2 "Resistor_SMD:R_0402_1005Metric_Pad0.72x0.64mm_HandSolder" V 2180 6600 50  0001 C CNN
 F 3 "~" H 2250 6600 50  0001 C CNN
 	1    2250 6600
@@
 F 0 "R4" V 2300 6850 50  0000 L CNN
 F 1 "1K" V 2300 6450 50  0000 L CNN
-F 2 "Resistor_SMD:R_0201_0603Metric_Pad0.64x0.40mm_HandSolder" V 2180 6700 50  0001 C CNN
+F 2 "Resistor_SMD:R_0402_1005Metric_Pad0.72x0.64mm_HandSolder" V 2180 6700 50  0001 C CNN
 F 3 "~" H 2250 6700 50  0001 C CNN
 	1    2250 6700
@@
 F 0 "C1" H 1400 6550 50  0000 C CNN
 F 1 "0.1 uF" H 1350 6650 50  0000 C CNN
-F 2 "Capacitor_SMD:C_0201_0603Metric_Pad0.64x0.40mm_HandSolder" H 1150 6550 50  0001 C CNN
+F 2 "Resistor_SMD:R_0402_1005Metric_Pad0.72x0.64mm_HandSolder" H 1150 6550 50  0001 C CNN
 F 3 "~" H 1150 6550 50  0001 C CNN
 	1    1150 6550
@@
 F 0 "R9" V 3850 6850 50  0000 L CNN
 F 1 "10K" V 3850 6450 50  0000 L CNN
-F 2 "Resistor_SMD:R_0201_0603Metric_Pad0.64x0.40mm_HandSolder" V 3730 6700 50  0001 C CNN
+F 2 "Resistor_SMD:R_0402_1005Metric_Pad0.72x0.64mm_HandSolder" V 3730 6700 50  0001 C CNN
 F 3 "~" H 3800 6700 50  0001 C CNN
 	1    3800 6700
@@
 F 0 "C3" H 4600 6600 50  0000 C CNN
 F 1 "10 uF" H 4550 6700 50  0000 C CNN
-F 2 "Capacitor_SMD:C_0201_0603Metric_Pad0.64x0.40mm_HandSolder" H 4350 6600 50  0001 C CNN
+F 2 "Resistor_SMD:R_0402_1005Metric_Pad0.72x0.64mm_HandSolder" H 4350 6600 50  0001 C CNN
 F 3 "~" H 4350 6600 50  0001 C CNN
 	1    4350 6600
@@
 F 0 "R12" H 5000 6700 50  0000 L CNN
 F 1 "1K" H 5000 6600 50  0000 L CNN
-F 2 "Resistor_SMD:R_0201_0603Metric_Pad0.64x0.40mm_HandSolder" V 4830 6600 50  0001 C CNN
+F 2 "Resistor_SMD:R_0402_1005Metric_Pad0.72x0.64mm_HandSolder" V 4830 6600 50  0001 C CNN
 F 3 "~" H 4900 6600 50  0001 C CNN
 	1    4900 6600
@@
 F 0 "C6" H 6700 6000 50  0000 C CNN
 F 1 "0.1 uF" H 6650 6100 50  0000 C CNN
-F 2 "Capacitor_SMD:C_0201_0603Metric_Pad0.64x0.40mm_HandSolder" H 6450 6000 50  0001 C CNN
+F 2 "Resistor_SMD:R_0402_1005Metric_Pad0.72x0.64mm_HandSolder" H 6450 6000 50  0001 C CNN
 F 3 "~" H 6450 6000 50  0001 C CNN
 	1    6450 6000
@@
 F 0 "R13" V 6850 5650 50  0000 L CNN
 F 1 "100" V 6850 5250 50  0000 L CNN
-F 2 "Resistor_SMD:R_0201_0603Metric_Pad0.64x0.40mm_HandSolder" V 6730 5500 50  0001 C CNN
+F 2 "Resistor_SMD:R_0402_1005Metric_Pad0.72x0.64mm_HandSolder" V 6730 5500 50  0001 C CNN
 F 3 "~" H 6800 5500 50  0001 C CNN
 	1    6800 5500
@@
 F 0 "R15" H 7850 2150 50  0000 C CNN
 F 1 "12K" H 7850 2050 50  0000 C CNN
-F 2 "Resistor_SMD:R_0201_0603Metric_Pad0.64x0.40mm_HandSolder" V 7630 2100 50  0001 C CNN
+F 2 "Resistor_SMD:R_0402_1005Metric_Pad0.72x0.64mm_HandSolder" V 7630 2100 50  0001 C CNN
 F 3 "~" H 7700 2100 50  0001 C CNN
 	1    7700 2100
@@
 F 0 "R14" H 7550 2150 50  0000 C CNN
 F 1 "12K" H 7550 2050 50  0000 C CNN
-F 2 "Resistor_SMD:R_0201_0603Metric_Pad0.64x0.40mm_HandSolder" V 7330 2100 50  0001 C CNN
+F 2 "Resistor_SMD:R_0402_1005Metric_Pad0.72x0.64mm_HandSolder" V 7330 2100 50  0001 C CNN
 F 3 "~" H 7400 2100 50  0001 C CNN
 	1    7400 2100
@@
 F 0 "C7" V 7000 2000 50  0000 C CNN
 F 1 "100 nF" V 6900 2000 50  0000 C CNN
-F 2 "Capacitor_SMD:C_0201_0603Metric_Pad0.64x0.40mm_HandSolder" H 6700 2000 50  0001 C CNN
+F 2 "Resistor_SMD:R_0402_1005Metric_Pad0.72x0.64mm_HandSolder" H 6700 2000 50  0001 C CNN
 F 3 "~" H 6700 2000 50  0001 C CNN
 	1    6700 2000
@@
 F 0 "R18" V 9450 2700 50  0000 C CNN
 F 1 "470" V 9450 2300 50  0000 C CNN
-F 2 "Resistor_SMD:R_0201_0603Metric_Pad0.64x0.40mm_HandSolder" V 9430 2500 50  0001 C CNN
+F 2 "Resistor_SMD:R_0402_1005Metric_Pad0.72x0.64mm_HandSolder" V 9430 2500 50  0001 C CNN
 F 3 "~" H 9500 2500 50  0001 C CNN
 	1    9500 2500
@@
 F 0 "R17" H 9550 3600 50  0000 C CNN
 F 1 "12K" H 9550 3500 50  0000 C CNN
-F 2 "Resistor_SMD:R_0201_0603Metric_Pad0.64x0.40mm_HandSolder" V 9330 3550 50  0001 C CNN
+F 2 "Resistor_SMD:R_0402_1005Metric_Pad0.72x0.64mm_HandSolder" V 9330 3550 50  0001 C CNN
 F 3 "~" H 9400 3550 50  0001 C CNN
 	1    9400 3550
@@
 F 0 "R19" H 10200 2850 50  0000 C CNN
 F 1 "12K" H 10200 2750 50  0000 C CNN
-F 2 "Resistor_SMD:R_0201_0603Metric_Pad0.64x0.40mm_HandSolder" V 9980 2800 50  0001 C CNN
+F 2 "Resistor_SMD:R_0402_1005Metric_Pad0.72x0.64mm_HandSolder" V 9980 2800 50  0001 C CNN
 F 3 "~" H 10050 2800 50  0001 C CNN
 	1    10050 2800
@@
 F 0 "R20" H 10500 2850 50  0000 C CNN
 F 1 "12K" H 10500 2750 50  0000 C CNN
-F 2 "Resistor_SMD:R_0201_0603Metric_Pad0.64x0.40mm_HandSolder" V 10280 2800 50  0001 C CNN
+F 2 "Resistor_SMD:R_0402_1005Metric_Pad0.72x0.64mm_HandSolder" V 10280 2800 50  0001 C CNN
 F 3 "~" H 10350 2800 50  0001 C CNN
 	1    10350 2800
@@
 F 0 "C8" H 8200 5550 50  0000 C CNN
 F 1 "0.1 uF" H 8150 5650 50  0000 C CNN
-F 2 "Capacitor_SMD:C_0201_0603Metric_Pad0.64x0.40mm_HandSolder" H 7950 5550 50  0001 C CNN
+F 2 "Resistor_SMD:R_0402_1005Metric_Pad0.72x0.64mm_HandSolder" H 7950 5550 50  0001 C CNN
 F 3 "~" H 7950 5550 50  0001 C CNN
 	1    7950 5550
@@
 F 0 "C9" H 8700 5950 50  0000 C CNN
 F 1 "0.1 uF" H 8650 6050 50  0000 C CNN
-F 2 "Capacitor_SMD:C_0201_0603Metric_Pad0.64x0.40mm_HandSolder" H 8450 5950 50  0001 C CNN
+F 2 "Resistor_SMD:R_0402_1005Metric_Pad0.72x0.64mm_HandSolder" H 8450 5950 50  0001 C CNN
 F 3 "~" H 8450 5950 50  0001 C CNN
 	1    8450 5950
@@
 F 0 "R16" H 8550 5550 50  0000 L CNN
 F 1 "100" H 8550 5450 50  0000 L CNN
-F 2 "Resistor_SMD:R_0201_0603Metric_Pad0.64x0.40mm_HandSolder" V 8380 5450 50  0001 C CNN
+F 2 "Resistor_SMD:R_0402_1005Metric_Pad0.72x0.64mm_HandSolder" V 8380 5450 50  0001 C CNN
 F 3 "~" H 8450 5450 50  0001 C CNN
 	1    8450 5450
@@
 F 0 "C10" H 10400 5700 50  0000 C CNN
 F 1 "0.1 uF" H 10350 5800 50  0000 C CNN
-F 2 "Capacitor_SMD:C_0201_0603Metric_Pad0.64x0.40mm_HandSolder" H 10150 5700 50  0001 C CNN
+F 2 "Resistor_SMD:R_0402_1005Metric_Pad0.72x0.64mm_HandSolder" H 10150 5700 50  0001 C CNN
 F 3 "~" H 10150 5700 50  0001 C CNN
 	1    10150 5700
